File: KiCad/noise-toy.kicad_sch (KiCad schematic)
At the start: 59 parts, among them J1 InputJack, J2 OutputJack, J3 Conn_02x20_PiZero, J4 Barrel_Jack_Switch, SW1 SWITCH_3PDT, SW2 SW_PUSH, SW3 SW_PUSH, SW4 SWITCH_INV, U1 MCP6002, U2 MCP3002

Commit message: Changed pcb attribution
Other:
- company: ElectroSmash.com -> Noise-Toy
- title: pedalpi.sch -> Noise-Toy
Changed lines of the file:
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@@
   (paper "A4")
   (title_block
-    (title "pedalpi.sch")
-    (date "2017-01-01")
-    (rev "rev. A")
-    (company "ElectroSmash.com")
+    (title "Noise-Toy")
+    (date "2023-09-11")
+    (rev "Rev 1")
+    (company "Noise-Toy")
+    (comment 1 "CC-BY ElectroSmash.com")
   )
   (junction (at 30.48 172.72) (diameter 0) (color 0 0 0 0)
